File: hardware/pico-breadboard.kicad_pcb (KiCad board)
At the start: 2 copper layers, 100 x 93 mm, 24 parts, among them J3 5V CONNECTOR, J4 GND CONNECTOR, J5 3.3V CONNECTOR, J6 Conn_01x20, J7 Conn_01x20, J8 SCREEN CONNECTOR, U1 Pico

Commit message: Add files via upload
Parts:
- BUTTON1, BUTTON2: footprint Button_Switch_THT:SW_PUSH_6mm -> Library:SW_PUSH_6mm
- BZ1: footprint Buzzer_Beeper:Buzzer_15x7.5RM7.6 -> Library:Buzzer_15x7.5RM7.6
- G*** (x3): footprint LOGO -> Library:LOGO
- J3, J4, J5, J8: footprint Connector_PinHeader_2.54mm:PinHeader_1x04_P2.54mm_Vertical -> Library:PinHeader_1x04_P2.54mm_Vertical
- J6, J7: footprint Connector_PinHeader_2.54mm:PinHeader_1x20_P2.54mm_Vertical -> Library:PinHeader_1x20_P2.54mm_Vertical
- LED1, LED2, LED3, LED4: footprint LED_THT:LED_D5.0mm -> Library:LED_D5.0mm
- R1, R2, R3, R4, R9: footprint Resistor_THT:R_Axial_DIN0204_L3.6mm_D1.6mm_P7.62mm_Horizontal -> Library:R_Axial_DIN0204_L3.6mm_D1.6mm_P7.62mm_Horizontal
- TR1: footprint Package_TO_SOT_THT:TO-92_Inline -> Library:TO-92_Inline
- U1: footprint RPi_Pico:RPi_Pico_SMD_TH -> Library:RPi_Pico_SMD_TH
- U2: footprint Custom:Breadboard -> Library:Breadboard
Routing:
- net +5V: track 170.9 -> 155.2 mm
Changed lines of the file:
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@@
 	(net 38 "/SW1")
 	(net 39 "/SW2")
-	(footprint "LED_THT:LED_D5.0mm"
+	(footprint "Library:LED_D5.0mm"
 		(layer "F.Cu")
 		(at 166.65 117.85 180)
@@
 			(pintype "passive")
 		)
-		(model "${KICAD8_3DMODEL_DIR}/LED_THT.3dshapes/LED_D5.0mm.wrl"
+		(model "${KIPRJMOD}/lib/Library.3dmodels/LED_D5.0mm.wrl"
 			(offset
-				(xyz 0 0 0)
+				(xyz 0 0 -3)
 			)
 			(scale
@@
 		)
 	)
-	(footprint "Buzzer_Beeper:Buzzer_15x7.5RM7.6"
+	(footprint "Library:Buzzer_15x7.5RM7.6"
 		(layer "F.Cu")
 		(at 162.7 103.8 180)
@@
 		(fp_circle
 			(center 3.8 0)
-			(end 11.4 0)
+			(end 9.8 0)
 			(stroke
 				(width 0.12)
@@
 		(fp_circle
 			(center 3.8 0)
-			(end 11.55 0)
+			(end 9.85 0)
 			(stroke
 				(width 0.05)
@@
 		(fp_circle
 			(center 3.8 0)
-			(end 11.3 0)
+			(end 9.8 0)
 			(stroke
 				(width 0.1)
@@
 			(pintype "passive")
 		)
-		(model "${KICAD8_3DMODEL_DIR}/Buzzer_Beeper.3dshapes/Buzzer_15x7.5RM7.6.wrl"
+		(model "${KIPRJMOD}/lib/Library.3dmodels/Buzzer_5V.STEP"
 			(offset
-				(xyz 0 0 0)
+				(xyz 3.8 0 0)
 			)
 			(scale
@@
 			)
 			(rotate
-				(xyz 0 0 0)
+				(xyz -90 0 0)
 			)
 		)
 	)
-	(footprint "Package_TO_SOT_THT:TO-92_Inline"
+	(footprint "Library:TO-92_Inline"
 		(layer "F.Cu")
 		(at 148.3 106.15 90)
@@
 			(pintype "passive")
 		)
-		(model "${KICAD8_3DMODEL_DIR}/Package_TO_SOT_THT.3dshapes/TO-92_Inline.wrl"
+		(model "${KIPRJMOD}/lib/Library.3dmodels/TO-92_Inline.wrl"
 			(offset
-				(xyz 0 0 0)
+				(xyz 0 0 -2.5)
 			)
 			(scale
@@
 		)
 	)
-	(footprint "LED_THT:LED_D5.0mm"
+	(footprint "Library:LED_D5.0mm"
 		(layer "F.Cu")
 		(at 142.65 117.85 180)
@@
 			(pintype "passive")
 		)
-		(model "${KICAD8_3DMODEL_DIR}/LED_THT.3dshapes/LED_D5.0mm.wrl"
+		(model "${KIPRJMOD}/lib/Library.3dmodels/LED_D5.0mm.wrl"
 			(offset
-				(xyz 0 0 0)
+				(xyz 0 0 -3)
 			)
 			(scale
@@
 		)
 	)
-	(footprint "Resistor_THT:R_Axial_DIN0204_L3.6mm_D1.6mm_P7.62mm_Horizontal"
+	(footprint "Library:R_Axial_DIN0204_L3.6mm_D1.6mm_P7.62mm_Horizontal"
 		(layer "F.Cu")
 		(at 181.65 121.85 90)
@@
 			(pintype "passive")
 		)
-		(model "${KICAD8_3DMODEL_DIR}/Resistor_THT.3dshapes/R_Axial_DIN0204_L3.6mm_D1.6mm_P7.62mm_Horizontal.wrl"
+		(model "${KIPRJMOD}/lib/Library.3dmodels/R_Axial_DIN0204_L3.6mm_D1.6mm_P7.62mm_Horizontal.wrl"
 			(offset
 				(xyz 0 0 0)
@@
 		)
 	)
-	(footprint "Resistor_THT:R_Axial_DIN0204_L3.6mm_D1.6mm_P7.62mm_Horizontal"
+	(footprint "Library:R_Axial_DIN0204_L3.6mm_D1.6mm_P7.62mm_Horizontal"
 		(layer "F.Cu")
 		(at 140.8 99.64 -90)
@@
 			(pintype "passive")
 		)
-		(model "${KICAD8_3DMODEL_DIR}/Resistor_THT.3dshapes/R_Axial_DIN0204_L3.6mm_D1.6mm_P7.62mm_Horizontal.wrl"
+		(model "${KIPRJMOD}/lib/Library.3dmodels/R_Axial_DIN0204_L3.6mm_D1.6mm_P7.62mm_Horizontal.wrl"
 			(offset
 				(xyz 0 0 0)
@@
 		)
 	)
-	(footprint "Button_Switch_THT:SW_PUSH_6mm"
+	(footprint "Library:SW_PUSH_6mm"
 		(layer "F.Cu")
 		(at 149.65 129.85 180)
@@
 			(pintype "passive")
 		)
-		(model "${KICAD8_3DMODEL_DIR}/Button_Switch_THT.3dshapes/SW_PUSH_6mm.wrl"
+		(model "${KIPRJMOD}/lib/Library.3dmodels/SW_PUSH_6mm.wrl"
 			(offset
 				(xyz 0 0 0)
@@
 		)
 	)
-	(footprint "Connector_PinHeader_2.54mm:PinHeader_1x20_P2.54mm_Vertical"
+	(footprint "Library:PinHeader_1x20_P2.54mm_Vertical"
 		(layer "F.Cu")
 		(at 87 97.85 90)
@@
 			(pintype "passive")
 		)
-		(model "${KICAD8_3DMODEL_DIR}/Connector_PinHeader_2.54mm.3dshapes/PinHeader_1x20_P2.54mm_Vertical.wrl"
+		(model "${KIPRJMOD}/lib/Library.3dmodels/PinHeader_1x20_P2.54mm_Vertical.wrl"
 			(offset
 				(xyz 0 0 0)
@@
 		)
 	)
-	(footprint "RPi_Pico:RPi_Pico_SMD_TH"
+	(footprint "Library:RPi_Pico_SMD_TH"
 		(layer "F.Cu")
 		(at 111.15 114.35 90)
@@
 			(pintype "unspecified")
 		)
-		(model "/home/rustem/Downloads/raspberry-pi-pico-w-pins-1.snapshot.4/PICO_PinsDown.STEP"
+		(model "${KIPRJMOD}/lib/Library.3dmodels/PICO_PinsDown.STEP"
 			(offset
 				(xyz -10.5 -25.5 3)
@@
 		)
 	)
-	(footprint "Connector_PinHeader_2.54mm:PinHeader_1x04_P2.54mm_Vertical"
+	(footprint "Library:PinHeader_1x04_P2.54mm_Vertical"
 		(layer "F.Cu")
 		(at 179.4 100.93)
@@
 			(pintype "passive")
 		)
-		(model "${KICAD8_3DMODEL_DIR}/Connector_PinHeader_2.54mm.3dshapes/PinHeader_1x04_P2.54mm_Vertical.wrl"
+		(model "${KIPRJMOD}/lib/Library.3dmodels/PinHeader_1x04_P2.54mm_Vertical.wrl"
 			(offset
 				(xyz 0 0 0)
@@
 		)
 	)
-	(footprint "LED_THT:LED_D5.0mm"
+	(footprint "Library:LED_D5.0mm"
 		(layer "F.Cu")
 		(at 178.65 117.85 180)
@@
 			(pintype "passive")
 		)
-		(model "${KICAD8_3DMODEL_DIR}/LED_THT.3dshapes/LED_D5.0mm.wrl"
+		(model "${KIPRJMOD}/lib/Library.3dmodels/LED_D5.0mm.wrl"
 			(offset
-				(xyz 0 0 0)
+				(xyz 0 0 -3)
 			)
 			(scale
@@
 		)
 	)
-	(footprint "Connector_PinHeader_2.54mm:PinHeader_1x04_P2.54mm_Vertical"
+	(footprint "Library:PinHeader_1x04_P2.54mm_Vertical"
 		(layer "F.Cu")
 		(at 91.65 82.85)
@@
 			(pintype "passive")
 		)
-		(model "${KICAD8_3DMODEL_DIR}/Connector_PinHeader_2.54mm.3dshapes/PinHeader_1x04_P2.54mm_Vertical.wrl"
+		(model "${KIPRJMOD}/lib/Library.3dmodels/PinHeader_1x04_P2.54mm_Vertical.wrl"
 			(offset
 				(xyz 0 0 0)
@@
 		)
 	)
-	(footprint "Button_Switch_THT:SW_PUSH_6mm"
+	(footprint "Library:SW_PUSH_6mm"
 		(layer "F.Cu")
 		(at 173.65 129.85 180)
@@
 			(pintype "passive")
 		)
-		(model "${KICAD8_3DMODEL_DIR}/Button_Switch_THT.3dshapes/SW_PUSH_6mm.wrl"
+		(model "${KIPRJMOD}/lib/Library.3dmodels/SW_PUSH_6mm.wrl"
 			(offset
 				(xyz 0 0 0)
@@
 		)
 	)
-	(footprint "Connector_PinHeader_2.54mm:PinHeader_1x20_P2.54mm_Vertical"
+	(footprint "Library:PinHeader_1x20_P2.54mm_Vertical"
 		(layer "F.Cu")
 		(at 87 130.85 90)
@@
 			(pintype "passive")
 		)
-		(model "${KICAD8_3DMODEL_DIR}/Connector_PinHeader_2.54mm.3dshapes/PinHeader_1x20_P2.54mm_Vertical.wrl"
+		(model "${KIPRJMOD}/lib/Library.3dmodels/PinHeader_1x20_P2.54mm_Vertical.wrl"
 			(offset
 				(xyz 0 0 0)
@@
 		)
 	)
-	(footprint "LED_THT:LED_D5.0mm"
+	(footprint "Library:LED_D5.0mm"
 		(layer "F.Cu")
 		(at 154.65 117.85 180)
@@
 			(pintype "passive")
 		)
-		(model "${KICAD8_3DMODEL_DIR}/LED_THT.3dshapes/LED_D5.0mm.wrl"
+		(model "${KIPRJMOD}/lib/Library.3dmodels/LED_D5.0mm.wrl"
 			(offset
-				(xyz 0 0 0)
+				(xyz 0 0 -3)
 			)
 			(scale
@@
 		)
 	)
-	(footprint "Connector_PinHeader_2.54mm:PinHeader_1x04_P2.54mm_Vertical"
+	(footprint "Library:PinHeader_1x04_P2.54mm_Vertical"
 		(layer "F.Cu")
 		(at 91.65 64.85)
@@
 			(pintype "passive")
 		)
-		(model "${KICAD8_3DMODEL_DIR}/Connector_PinHeader_2.54mm.3dshapes/PinHeader_1x04_P2.54mm_Vertical.wrl"
+		(model "${KIPRJMOD}/lib/Library.3dmodels/PinHeader_1x04_P2.54mm_Vertical.wrl"
 			(offset
 				(xyz 0 0 0)
@@
 		)
 	)
-	(footprint "Custom:Breadboard"
+	(footprint "Library:Breadboard"
 		(layer "F.Cu")
 		(at 98.65 40.85)
@@
 			)
 		)
-		(model "/home/rustem/Downloads/half-breadboard-1.snapshot.3/HalfBreadboard.STEP"
+		(model "${KIPRJMOD}/lib/Library.3dmodels/HalfBreadboard.STEP"
 			(offset
 				(xyz 43 14.5 5)
@@
 		)
 	)
-	(footprint "Resistor_THT:R_Axial_DIN0204_L3.6mm_D1.6mm_P7.62mm_Horizontal"
+	(footprint "Library:R_Axial_DIN0204_L3.6mm_D1.6mm_P7.62mm_Horizontal"
 		(layer "F.Cu")
 		(at 169.65 121.85 90)
@@
 			(pintype "passive")
 		)
-		(model "${KICAD8_3DMODEL_DIR}/Resistor_THT.3dshapes/R_Axial_DIN0204_L3.6mm_D1.6mm_P7.62mm_Horizontal.wrl"
+		(model "${KIPRJMOD}/lib/Library.3dmodels/R_Axial_DIN0204_L3.6mm_D1.6mm_P7.62mm_Horizontal.wrl"
 			(offset
 				(xyz 0 0 0)
@@
 		)
 	)
-	(footprint "Connector_PinHeader_2.54mm:PinHeader_1x04_P2.54mm_Vertical"
+	(footprint "Library:PinHeader_1x04_P2.54mm_Vertical"
 		(layer "F.Cu")
 		(at 91.65 46.85)
@@
 			(pintype "passive")
 		)
-		(model "${KICAD8_3DMODEL_DIR}/Connector_PinHeader_2.54mm.3dshapes/PinHeader_1x04_P2.54mm_Vertical.wrl"
+		(model "${KIPRJMOD}/lib/Library.3dmodels/PinHeader_1x04_P2.54mm_Vertical.wrl"
 			(offset
 				(xyz 0 0 0)
@@
 		)
 	)
-	(footprint "Resistor_THT:R_Axial_DIN0204_L3.6mm_D1.6mm_P7.62mm_Horizontal"
+	(footprint "Library:R_Axial_DIN0204_L3.6mm_D1.6mm_P7.62mm_Horizontal"
 		(layer "F.Cu")
 		(at 157.65 121.85 90)
@@
 			(pintype "passive")
 		)
-		(model "${KICAD8_3DMODEL_DIR}/Resistor_THT.3dshapes/R_Axial_DIN0204_L3.6mm_D1.6mm_P7.62mm_Horizontal.wrl"
+		(model "${KIPRJMOD}/lib/Library.3dmodels/R_Axial_DIN0204_L3.6mm_D1.6mm_P7.62mm_Horizontal.wrl"
 			(offset
 				(xyz 0 0 0)
@@
 		)
 	)
-	(footprint "Resistor_THT:R_Axial_DIN0204_L3.6mm_D1.6mm_P7.62mm_Horizontal"
+	(footprint "Library:R_Axial_DIN0204_L3.6mm_D1.6mm_P7.62mm_Horizontal"
 		(layer "F.Cu")
 		(at 145.65 121.85 90)
@@
 			(pintype "passive")
 		)
-		(model "${KICAD8_3DMODEL_DIR}/Resistor_THT.3dshapes/R_Axial_DIN0204_L3.6mm_D1.6mm_P7.62mm_Horizontal.wrl"
+		(model "${KIPRJMOD}/lib/Library.3dmodels/R_Axial_DIN0204_L3.6mm_D1.6mm_P7.62mm_Horizontal.wrl"
 			(offset
 				(xyz 0 0 0)
@@
 		)
 	)
-	(footprint "LOGO"
+	(footprint "Library:LOGO"
 		(layer "B.Cu")
 		(at 145.817523 51.243196 180)
@@
 		)
 	)
-	(footprint "LOGO"
+	(footprint "Library:LOGO"
 		(layer "B.Cu")
 		(at 104 86.9 180)
@@
 		)
 	)
-	(footprint "LOGO"
+	(footprint "Library:LOGO"
 		(layer "B.Cu")
 		(at 102.35 50.95 180)
@@
 	)
 	(segment
-		(start 132.6 46.85)
-		(end 162.7 76.95)
-		(width 1.5)
-		(layer "F.Cu")
-		(net 12)
-	)
-	(segment
-		(start 162.7 76.95)
-		(end 162.7 103.8)
+		(start 91.65 46.85)
+		(end 105.75 46.85)
 		(width 1.5)
 		(layer "F.Cu")
@@
 	)
 	(segment
-		(start 91.65 46.85)
-		(end 132.6 46.85)
+		(start 105.75 46.85)
+		(end 162.7 103.8)
 		(width 1.5)
 		(layer "F.Cu")
