File: hardware/pico-breadboard.kicad_sch (KiCad schematic)
At the start: 21 parts, among them J3 5V CONNECTOR, J4 GND CONNECTOR, J5 3.3V CONNECTOR, J6 Conn_01x20, J7 Conn_01x20, J8 SCREEN CONNECTOR, U1 Pico

Commit message: Add files via upload
Parts:
- BUTTON1, BUTTON2: symbol Switch:SW_SPST -> Library:SW_SPST
- BZ1: symbol Device:Buzzer -> Library:Buzzer
- J3, J4, J5, J8: symbol Connector_Generic:Conn_01x04 -> Library:Conn_01x04
- J6, J7: symbol Connector_Generic:Conn_01x20 -> Library:Conn_01x20
- LED1, LED2, LED3, LED4: symbol Device:LED -> Library:LED
- R1, R2, R3, R4, R9: symbol Device:R_US -> Library:R_US
- TR1: symbol Transistor_BJT:BC517 -> Library:BC517
- U1: symbol RPi_Pico:Pico -> Library:Pico
- U2: symbol 000_customSymbols:Breadboard -> Library:Breadboard
Other:
- note added: "CONNECTORS"
Changed lines of the file:
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@@
 		)
 	)
+	(text "CONNECTORS\n"
+		(exclude_from_sim no)
+		(at 165.608 25.908 0)
+		(effects
+			(font
+				(size 1.27 1.27)
+			)
+		)
+	)
 	(text "LED"
 		(exclude_from_sim no)
@@
 	)
 	(symbol
-		(lib_id "power:+5V")
+		(lib_id "Library:+5V")
 		(at 46.99 43.18 0)
 		(unit 1)
@@
 	)
 	(symbol
-		(lib_id "power:+5V")
+		(lib_id "Library:+5V")
 		(at 190.5 72.39 180)
 		(unit 1)
@@
 	)
 	(symbol
-		(lib_id "power:+3.3V")
+		(lib_id "Library:+3.3V")
 		(at 185.42 44.45 270)
 		(unit 1)
@@
 	)
 	(symbol
-		(lib_id "Switch:SW_SPST")
+		(lib_id "Library:SW_SPST")
 		(at 125.73 49.53 0)
 		(unit 1)
@@
 	)
 	(symbol
-		(lib_id "Connector_Generic:Conn_01x20")
+		(lib_id "Library:Conn_01x20")
 		(at 129.54 123.19 0)
 		(unit 1)
@@
 	)
 	(symbol
-		(lib_id "power:PWR_FLAG")
+		(lib_id "Library:PWR_FLAG")
 		(at 46.99 43.18 90)
 		(unit 1)
@@
 	)
 	(symbol
-		(lib_id "power:GND")
+		(lib_id "Library:GND")
 		(at 132.08 143.51 90)
 		(unit 1)
@@
 	)
 	(symbol
-		(lib_id "Connector_Generic:Conn_01x04")
+		(lib_id "Library:Conn_01x04")
 		(at 181.61 118.11 0)
 		(mirror y)
@@
 	)
 	(symbol
-		(lib_id "power:PWR_FLAG")
+		(lib_id "Library:PWR_FLAG")
 		(at 96.52 81.28 180)
 		(unit 1)
@@
 	)
 	(symbol
-		(lib_id "Connector_Generic:Conn_01x04")
+		(lib_id "Library:Conn_01x04")
 		(at 181.61 67.31 0)
 		(mirror y)
@@
 	)
 	(symbol
-		(lib_id "power:GND")
+		(lib_id "Library:GND")
 		(at 52.07 118.11 270)
 		(unit 1)
@@
 	)
 	(symbol
-		(lib_id "power:PWR_FLAG")
+		(lib_id "Library:PWR_FLAG")
 		(at 128.27 81.28 180)
 		(unit 1)
@@
 	)
 	(symbol
-		(lib_id "power:GND")
+		(lib_id "Library:GND")
 		(at 52.07 143.51 270)
 		(unit 1)
@@
 	)
 	(symbol
-		(lib_id "Device:Buzzer")
+		(lib_id "Library:Buzzer")
 		(at 49.53 49.53 0)
 		(unit 1)
@@
 	)
 	(symbol
-		(lib_id "Transistor_BJT:BC517")
+		(lib_id "Library:BC517")
 		(at 44.45 62.23 0)
 		(unit 1)
@@
 	)
 	(symbol
-		(lib_id "power:GND")
+		(lib_id "Library:GND")
 		(at 52.07 105.41 270)
 		(unit 1)
@@
 	)
 	(symbol
-		(lib_id "power:GND")
+		(lib_id "Library:GND")
 		(at 104.14 80.01 0)
 		(unit 1)
@@
 	)
 	(symbol
-		(lib_id "Connector_Generic:Conn_01x20")
+		(lib_id "Library:Conn_01x20")
 		(at 55.88 123.19 0)
 		(mirror y)
@@
 	)
 	(symbol
-		(lib_id "RPi_Pico:Pico")
+		(lib_id "Library:Pico")
 		(at 92.71 124.46 0)
 		(unit 1)
@@
 	)
 	(symbol
-		(lib_id "Device:R_US")
+		(lib_id "Library:R_US")
 		(at 35.56 62.23 90)
 		(unit 1)
@@
 	)
 	(symbol
-		(lib_id "Device:LED")
+		(lib_id "Library:LED")
 		(at 87.63 62.23 180)
 		(unit 1)
@@
 	)
 	(symbol
-		(lib_id "power:GND")
+		(lib_id "Library:GND")
 		(at 133.35 105.41 90)
 		(unit 1)
@@
 	)
 	(symbol
-		(lib_id "power:GND")
+		(lib_id "Library:GND")
 		(at 52.07 130.81 270)
 		(unit 1)
@@
 	)
 	(symbol
-		(lib_id "Device:R_US")
+		(lib_id "Library:R_US")
 		(at 97.79 36.83 90)
 		(unit 1)
@@
 	)
 	(symbol
-		(lib_id "000_customSymbols:Breadboard")
+		(lib_id "Library:Breadboard")
 		(at 181.61 144.78 0)
 		(unit 1)
@@
 	)
 	(symbol
-		(lib_id "power:+3.3V")
+		(lib_id "Library:+3.3V")
 		(at 133.35 110.49 270)
 		(unit 1)
@@
 	)
 	(symbol
-		(lib_id "Connector_Generic:Conn_01x04")
+		(lib_id "Library:Conn_01x04")
 		(at 180.34 41.91 0)
 		(mirror y)
@@
 	)
 	(symbol
-		(lib_id "Connector_Generic:Conn_01x04")
+		(lib_id "Library:Conn_01x04")
 		(at 181.61 93.98 0)
 		(mirror y)
@@
 	)
 	(symbol
-		(lib_id "Device:R_US")
+		(lib_id "Library:R_US")
 		(at 97.79 62.23 90)
 		(unit 1)
@@
 	)
 	(symbol
-		(lib_id "Device:R_US")
+		(lib_id "Library:R_US")
 		(at 97.79 49.53 90)
 		(unit 1)
@@
 	)
 	(symbol
-		(lib_id "power:GND")
+		(lib_id "Library:GND")
 		(at 133.35 130.81 90)
 		(unit 1)
@@
 	)
 	(symbol
-		(lib_id "power:+3.3V")
+		(lib_id "Library:+3.3V")
 		(at 118.11 80.01 180)
 		(unit 1)
@@
 	)
 	(symbol
-		(lib_id "power:+3.3V")
+		(lib_id "Library:+3.3V")
 		(at 190.5 99.06 180)
 		(unit 1)
@@
 	)
 	(symbol
-		(lib_id "Switch:SW_SPST")
+		(lib_id "Library:SW_SPST")
 		(at 125.73 36.83 0)
 		(unit 1)
@@
 	)
 	(symbol
-		(lib_id "power:GND")
+		(lib_id "Library:GND")
 		(at 190.5 123.19 0)
 		(unit 1)
@@
 	)
 	(symbol
-		(lib_id "Device:LED")
+		(lib_id "Library:LED")
 		(at 87.63 74.93 180)
 		(unit 1)
@@
 	)
 	(symbol
-		(lib_id "power:GND")
+		(lib_id "Library:GND")
 		(at 185.42 46.99 90)
 		(unit 1)
@@
 	)
 	(symbol
-		(lib_id "Device:R_US")
+		(lib_id "Library:R_US")
 		(at 97.79 74.93 90)
 		(unit 1)
@@
 	)
 	(symbol
-		(lib_id "power:GND")
+		(lib_id "Library:GND")
 		(at 46.99 72.39 0)
 		(unit 1)
@@
 	)
 	(symbol
-		(lib_id "Device:LED")
+		(lib_id "Library:LED")
 		(at 87.63 49.53 180)
 		(unit 1)
@@
 	)
 	(symbol
-		(lib_id "power:GND")
+		(lib_id "Library:GND")
 		(at 133.35 118.11 90)
 		(unit 1)
@@
 	)
 	(symbol
-		(lib_id "power:+5V")
+		(lib_id "Library:+5V")
 		(at 133.35 100.33 270)
 		(unit 1)
@@
 	)
 	(symbol
-		(lib_id "Device:LED")
+		(lib_id "Library:LED")
 		(at 87.63 36.83 180)
 		(unit 1)

Commit message: minor changes
Parts:
- renumbered U2 to BREADBOARD
Changed lines of the file:
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@@
 		(on_board yes)
 		(dnp no)
-		(property "Reference" "U2"
-			(at 179.578 144.78 0)
+		(property "Reference" "BREADBOARD"
+			(at 174.752 144.526 0)
 			(effects
 				(font
@@
 			(project ""
 				(path "/8dc432d0-705f-48a2-b043-b7130b9baf7d"
-					(reference "U2")
+					(reference "BREADBOARD")
 					(unit 1)
 				)
