File: v2/hardware/pico-breadboard.kicad_sch (KiCad schematic)
At the start: 21 parts, among them J3 5V CONNECTOR, J4 GND CONNECTOR, J5 3.3V CONNECTOR, J6 Conn_01x20, J7 Conn_01x20, J8 SCREEN CONNECTOR, U1 Pico

Commit message: v2 updated
Parts:
- removed BREADBOARD: ~, Custom:Breadboard, symbol Library:Breadboard
- removed BUTTON1, BUTTON2: SW_SPST, Button_Switch_THT:SW_PUSH_6mm, symbol Library:SW_SPST
- removed J6, J7: Conn_01x20, Connector_PinHeader_2.54mm:PinHeader_1x20_P2.54mm_Vertical, symbol Library:Conn_01x20
- removed TR1: BC517, Package_TO_SOT_THT:TO-92_Inline, symbol Library:BC517
- added FID1, FID2, FID3, FID4: Fiducial, Fiducial:Fiducial_1mm_Mask2mm, symbol Mechanical:Fiducial
- added H1, H2, H3, H4: MountingHole, MountingHole:MountingHole_3mm, symbol Mechanical:MountingHole
- added J1: Conn_01x05, Connector_PinHeader_2.54mm:PinHeader_1x05_P2.54mm_Vertical, symbol Connector_Generic:Conn_01x05
- added J10: MPU6050 CONNECTOR, Connector_PinHeader_2.54mm:PinHeader_1x04_P2.54mm_Vertical, symbol Library:Conn_01x04
- added J11, J12, J9: Conn_01x03, Connector_PinHeader_2.54mm:PinHeader_1x03_P2.54mm_Vertical, symbol Connector_Generic:Conn_01x03
- added J2: LED, Connector_PinHeader_2.54mm:PinHeader_1x04_P2.54mm_Vertical, symbol Library:Conn_01x04
- added J6: Conn_01x12, Connector_PinHeader_2.54mm:PinHeader_1x12_P2.54mm_Vertical, symbol Connector_Generic:Conn_01x12
- added J7: Conn_01x11, Connector_PinHeader_2.54mm:PinHeader_1x11_P2.54mm_Vertical, symbol Connector_Generic:Conn_01x11
- added Q1: BC817, Package_TO_SOT_SMD:SOT-23, symbol Library:BC817
- added RV1: R_Potentiometer, Library:Potentiometer_Omeg_PC16BU_Horizontal, symbol Library:R_Potentiometer
- added SW1, SW2, SW3, SW4: SW_SPST, Library:SW_SPST_PTS810, symbol Library:SW_SPST
- added SW5: RotaryEncoder_Switch_MP, Library:RotaryEncoder_Alps_EC11E-Switch_Vertical_H20mm, symbol Library:RotaryEncoder_Switch_MP
- added U2: ~, Library:Breadboard, symbol Library:Breadboard
- BZ1: footprint Buzzer_Beeper:Buzzer_15x7.5RM7.6 -> Library:Buzzer_12mm7.6
- LED1, LED2, LED3, LED4: footprint LED_THT:LED_D5.0mm -> LED_SMD:LED_0603_1608Metric
- R1, R2, R3, R4, R9: footprint Resistor_THT:R_Axial_DIN0204_L3.6mm_D1.6mm_P7.62mm_Horizontal -> Resistor_SMD:R_0402_1005Metric
Connections:
- net +3.3V: now also J8.2 (Pin_2), J10.1 (Pin_1), RV1.3, SW1.1 (A), SW2.1 (A), SW3.1 (A), SW4.1 (A), SW5.S1; no longer J8.3 (Pin_3)
- net +5V: now also U1.39 (VSYS), J11.2 (Pin_2), J12.3 (Pin_3), J9.2 (Pin_2); no longer U1.40 (VBUS)
- net BUZZER: now also U1.12 (GPIO9); no longer U1.24 (GPIO18)
- net GND: now also J8.1 (Pin_1), J10.2 (Pin_2), J11.1 (Pin_1), J12.1 (Pin_1), J9.1 (Pin_1), Q1.2 (E), RV1.1, SW5.C; no longer J8.4 (Pin_4)
- net LED1: now also J2.1 (Pin_1); no longer U1.19 (GPIO14)
- net LED2: now also J2.2 (Pin_2); no longer U1.20 (GPIO15)
- net LED3: now also J2.3 (Pin_3); no longer U1.21 (GPIO16)
- net LED4: now also J2.4 (Pin_4); no longer U1.22 (GPIO17)
- net SW1: now also J1.1 (Pin_1), SW1.2 (B); no longer U1.17 (GPIO13)
- net SW2: now also J1.2 (Pin_2), SW2.2 (B); no longer U1.16 (GPIO12)
- net GPIO26: now reaches U1.31 (GPIO26_ADC0)
- net GPIO26: now also J7.3 (Pin_3), RV1.2
- net GPIO22: now reaches U1.29 (GPIO22)
- net GPIO22: now also J7.4 (Pin_4)
- net GPIO19: now reaches U1.25 (GPIO19)
- net GPIO19: now also J7.7 (Pin_7)
- net GPIO28: now reaches U1.34 (GPIO28_ADC2)
- net GPIO28: now also J7.1 (Pin_1)
- net GPIO27: now reaches U1.32 (GPIO27_ADC1)
- net GPIO27: now also J7.2 (Pin_2)
- net at BZ1.2 (-): now also Q1.3 (C)
- net at R9.2: now also Q1.1 (B)
- net GPIO0: now reaches U1.1 (GPIO0)
- net GPIO0: now also J12.2 (Pin_2), J6.1 (Pin_1)
- net GPIO7: now reaches U1.10 (GPIO7)
- net GPIO7: now also J6.8 (Pin_8)
- net GPIO8: now reaches U1.11 (GPIO8)
- net GPIO8: now also J6.9 (Pin_9)
- net GPIO10: now reaches U1.14 (GPIO10)
- net GPIO10: now also J6.10 (Pin_10), J9.3 (Pin_3)
- net GPIO11: now reaches U1.15 (GPIO11)
- net GPIO11: now also J11.3 (Pin_3), J6.11 (Pin_11)
- net GPIO1: now reaches U1.2 (GPIO1)
- net GPIO1: now also J6.2 (Pin_2)
- net GPIO2: now reaches U1.4 (GPIO2)
- net GPIO2: now also J6.3 (Pin_3)
- net GPIO3: now reaches U1.5 (GPIO3)
- net GPIO3: now also J6.4 (Pin_4)
- net GPIO4: now reaches U1.6 (GPIO4)
- net GPIO4: now also J6.5 (Pin_5)
- net GPIO5: now reaches U1.7 (GPIO5)
- net GPIO5: now also J6.6 (Pin_6)
- net GPIO6: now reaches U1.9 (GPIO6)
- net GPIO6: now also J6.7 (Pin_7)
- net SCL renamed GPIO21
- net GPIO21: now also J7.5 (Pin_5); no longer J8.2 (Pin_2)
- net SDA renamed GPIO20
- net GPIO20: now also J7.6 (Pin_6); no longer J8.1 (Pin_1)
- new net A: SW5.A, U1.19 (GPIO14)
- new net B: SW5.B, U1.20 (GPIO15)
- new net GPIO12: J10.4 (Pin_4), J6.12 (Pin_12), J8.4 (Pin_4), U1.16 (GPIO12)
- new net GPIO13: J10.3 (Pin_3), J7.11 (Pin_11), J8.3 (Pin_3), U1.17 (GPIO13)
- new net GPIO16: J7.10 (Pin_10), U1.21 (GPIO16)
- new net GPIO17: J7.9 (Pin_9), U1.22 (GPIO17)
- new net GPIO18: J7.8 (Pin_8), U1.24 (GPIO18)
- new net SW3: J1.3 (Pin_3), SW3.2 (B)
- new net SW4: J1.4 (Pin_4), SW4.2 (B)
- new net SW5: J1.5 (Pin_5), SW5.S2
- no-connect marks 0 -> 4

Commit message: update
Parts:
- U2: value ~ -> BREADBOARD
Other:
- moved on the sheet: FID1, FID2, FID3, FID4, H1, H2, H3, H4, J1, J10, J11, J12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

Commit message: update
Parts:
- FID1, FID2, FID3, FID4: footprint Fiducial:Fiducial_1mm_Mask2mm -> Library:Fiducial_1mm_Mask2mm; symbol Mechanical:Fiducial -> Library:Fiducial
- H1, H2, H3, H4: footprint MountingHole:MountingHole_3mm -> Library:MountingHole_3mm; symbol Mechanical:MountingHole -> Library:MountingHole
- J1: footprint Connector_PinHeader_2.54mm:PinHeader_1x05_P2.54mm_Vertical -> Library:PinHeader_1x05_P2.54mm_Vertical; symbol Connector_Generic:Conn_01x05 -> Library:Conn_01x05
- J10, J2, J3, J4, J5, J8: footprint Connector_PinHeader_2.54mm:PinHeader_1x04_P2.54mm_Vertical -> Library:PinHeader_1x04_P2.54mm_Vertical
- J11, J12, J9: footprint Connector_PinHeader_2.54mm:PinHeader_1x03_P2.54mm_Vertical -> Library:PinHeader_1x03_P2.54mm_Vertical; symbol Connector_Generic:Conn_01x03 -> Library:Conn_01x03
- J6: footprint Connector_PinHeader_2.54mm:PinHeader_1x12_P2.54mm_Vertical -> Library:PinHeader_1x12_P2.54mm_Vertical; symbol Connector_Generic:Conn_01x12 -> Library:Conn_01x12
- J7: footprint Connector_PinHeader_2.54mm:PinHeader_1x11_P2.54mm_Vertical -> Library:PinHeader_1x11_P2.54mm_Vertical; symbol Connector_Generic:Conn_01x11 -> Library:Conn_01x11
- LED1, LED2, LED3, LED4: footprint LED_SMD:LED_0603_1608Metric -> Library:LED_0603_1608Metric
- Q1: footprint Package_TO_SOT_SMD:SOT-23 -> Library:SOT-23
- R1, R2, R3, R4, R9: footprint Resistor_SMD:R_0402_1005Metric -> Library:R_0402_1005Metric
- U1: footprint RPi_Pico:RPi_Pico_SMD_TH -> Library:RPi_Pico_SMD_TH
Changed lines of the file:
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@@
 	)
 	(symbol
-		(lib_id "Mechanical:Fiducial")
+		(lib_id "Library:Fiducial")
 		(at 228.6 146.05 0)
 		(unit 1)
@@
 			)
 		)
-		(property "Footprint" "Fiducial:Fiducial_1mm_Mask2mm"
+		(property "Footprint" "Library:Fiducial_1mm_Mask2mm"
 			(at 228.6 146.05 0)
 			(effects
@@
 	)
 	(symbol
-		(lib_id "Connector_Generic:Conn_01x11")
+		(lib_id "Library:Conn_01x11")
 		(at 218.44 120.65 0)
 		(mirror y)
@@
 			)
 		)
-		(property "Footprint" "Connector_PinHeader_2.54mm:PinHeader_1x11_P2.54mm_Vertical"
+		(property "Footprint" "Library:PinHeader_1x11_P2.54mm_Vertical"
 			(at 218.44 120.65 0)
 			(effects
@@
 	)
 	(symbol
-		(lib_id "Mechanical:Fiducial")
+		(lib_id "Library:Fiducial")
 		(at 228.6 152.4 0)
 		(unit 1)
@@
 			)
 		)
-		(property "Footprint" "Fiducial:Fiducial_1mm_Mask2mm"
+		(property "Footprint" "Library:Fiducial_1mm_Mask2mm"
 			(at 228.6 152.4 0)
 			(effects
@@
 			)
 		)
-		(property "Footprint" "Connector_PinHeader_2.54mm:PinHeader_1x04_P2.54mm_Vertical"
+		(property "Footprint" "Library:PinHeader_1x04_P2.54mm_Vertical"
 			(at 255.27 43.18 0)
 			(effects
@@
 			)
 		)
-		(property "Footprint" "Connector_PinHeader_2.54mm:PinHeader_1x04_P2.54mm_Vertical"
+		(property "Footprint" "Library:PinHeader_1x04_P2.54mm_Vertical"
 			(at 223.52 63.5 0)
 			(effects
@@
 			)
 		)
-		(property "Footprint" "Connector_PinHeader_2.54mm:PinHeader_1x04_P2.54mm_Vertical"
+		(property "Footprint" "Library:PinHeader_1x04_P2.54mm_Vertical"
 			(at 180.34 44.45 0)
 			(effects
@@
 	)
 	(symbol
-		(lib_id "Mechanical:MountingHole")
+		(lib_id "Library:MountingHole")
 		(at 184.15 152.4 0)
 		(unit 1)
@@
 			)
 		)
-		(property "Footprint" "MountingHole:MountingHole_3mm"
+		(property "Footprint" "Library:MountingHole_3mm"
 			(at 184.15 152.4 0)
 			(effects
@@
 			)
 		)
-		(property "Footprint" "Connector_PinHeader_2.54mm:PinHeader_1x04_P2.54mm_Vertical"
+		(property "Footprint" "Library:PinHeader_1x04_P2.54mm_Vertical"
 			(at 181.61 63.5 0)
 			(effects
@@
 			)
 		)
-		(property "Footprint" "Connector_PinHeader_2.54mm:PinHeader_1x04_P2.54mm_Vertical"
+		(property "Footprint" "Library:PinHeader_1x04_P2.54mm_Vertical"
 			(at 223.52 44.45 0)
 			(effects
@@
 			)
 		)
-		(property "Footprint" "RPi_Pico:RPi_Pico_SMD_TH"
+		(property "Footprint" "Library:RPi_Pico_SMD_TH"
 			(at 59.69 123.19 90)
 			(effects
@@
 			)
 		)
-		(property "Footprint" "Resistor_SMD:R_0402_1005Metric"
+		(property "Footprint" "Library:R_0402_1005Metric"
 			(at 35.814 61.214 90)
 			(effects
@@
 	)
 	(symbol
-		(lib_id "Connector_Generic:Conn_01x03")
+		(lib_id "Library:Conn_01x03")
 		(at 181.61 86.36 0)
 		(mirror y)
@@
 			)
 		)
-		(property "Footprint" "Connector_PinHeader_2.54mm:PinHeader_1x03_P2.54mm_Vertical"
+		(property "Footprint" "Library:PinHeader_1x03_P2.54mm_Vertical"
 			(at 181.61 86.36 0)
 			(effects
@@
 			)
 		)
-		(property "Footprint" "LED_SMD:LED_0603_1608Metric"
+		(property "Footprint" "Library:LED_0603_1608Metric"
 			(at 87.63 62.23 0)
 			(effects
@@
 	)
 	(symbol
-		(lib_id "Mechanical:Fiducial")
+		(lib_id "Library:Fiducial")
 		(at 241.3 152.4 0)
 		(unit 1)
@@
 			)
 		)
-		(property "Footprint" "Fiducial:Fiducial_1mm_Mask2mm"
+		(property "Footprint" "Library:Fiducial_1mm_Mask2mm"
 			(at 241.3 152.4 0)
 			(effects
@@
 	)
 	(symbol
-		(lib_id "Connector_Generic:Conn_01x03")
+		(lib_id "Library:Conn_01x03")
 		(at 255.27 87.63 0)
 		(mirror y)
@@
 			)
 		)
-		(property "Footprint" "Connector_PinHeader_2.54mm:PinHeader_1x03_P2.54mm_Vertical"
+		(property "Footprint" "Library:PinHeader_1x03_P2.54mm_Vertical"
 			(at 255.27 87.63 0)
 			(effects
@@
 			)
 		)
-		(property "Footprint" "Resistor_SMD:R_0402_1005Metric"
+		(property "Footprint" "Library:R_0402_1005Metric"
 			(at 98.044 35.814 90)
 			(effects
@@
 	)
 	(symbol
-		(lib_id "Mechanical:MountingHole")
+		(lib_id "Library:MountingHole")
 		(at 203.2 152.4 0)
 		(unit 1)
@@
 			)
 		)
-		(property "Footprint" "MountingHole:MountingHole_3mm"
+		(property "Footprint" "Library:MountingHole_3mm"
 			(at 203.2 152.4 0)
 			(effects
@@
 	)
 	(symbol
-		(lib_id "Connector_Generic:Conn_01x05")
+		(lib_id "Library:Conn_01x05")
 		(at 254 115.57 0)
 		(mirror y)
@@
 			)
 		)
-		(property "Footprint" "Connector_PinHeader_2.54mm:PinHeader_1x05_P2.54mm_Vertical"
+		(property "Footprint" "Library:PinHeader_1x05_P2.54mm_Vertical"
 			(at 254 115.57 0)
 			(effects
@@
 			)
 		)
-		(property "Footprint" "Connector_PinHeader_2.54mm:PinHeader_1x04_P2.54mm_Vertical"
+		(property "Footprint" "Library:PinHeader_1x04_P2.54mm_Vertical"
 			(at 255.27 62.23 0)
 			(effects
@@
 			)
 		)
-		(property "Footprint" "Resistor_SMD:R_0402_1005Metric"
+		(property "Footprint" "Library:R_0402_1005Metric"
 			(at 98.044 61.214 90)
 			(effects
@@
 	)
 	(symbol
-		(lib_id "Connector_Generic:Conn_01x03")
+		(lib_id "Library:Conn_01x03")
 		(at 218.44 87.63 0)
 		(mirror y)
@@
 			)
 		)
-		(property "Footprint" "Connector_PinHeader_2.54mm:PinHeader_1x03_P2.54mm_Vertical"
+		(property "Footprint" "Library:PinHeader_1x03_P2.54mm_Vertical"
 			(at 218.44 87.63 0)
 			(effects
@@
 			)
 		)
-		(property "Footprint" "Resistor_SMD:R_0402_1005Metric"
+		(property "Footprint" "Library:R_0402_1005Metric"
 			(at 98.044 48.514 90)
 			(effects
@@
 	)
 	(symbol
-		(lib_id "Connector_Generic:Conn_01x12")
+		(lib_id "Library:Conn_01x12")
 		(at 180.34 121.92 0)
 		(unit 1)
@@
 			)
 		)
-		(property "Footprint" "Connector_PinHeader_2.54mm:PinHeader_1x12_P2.54mm_Vertical"
+		(property "Footprint" "Library:PinHeader_1x12_P2.54mm_Vertical"
 			(at 180.34 121.92 0)
 			(effects
@@
 	)
 	(symbol
-		(lib_id "Mechanical:MountingHole")
+		(lib_id "Library:MountingHole")
 		(at 184.15 146.05 0)
 		(unit 1)
@@
 			)
 		)
-		(property "Footprint" "MountingHole:MountingHole_3mm"
+		(property "Footprint" "Library:MountingHole_3mm"
 			(at 184.15 146.05 0)
 			(effects
@@
 	)
 	(symbol
-		(lib_id "Mechanical:MountingHole")
+		(lib_id "Library:MountingHole")
 		(at 203.2 146.05 0)
 		(unit 1)
@@
 			)
 		)
-		(property "Footprint" "MountingHole:MountingHole_3mm"
+		(property "Footprint" "Library:MountingHole_3mm"
 			(at 203.2 146.05 0)
 			(effects
@@
 	)
 	(symbol
-		(lib_id "Mechanical:Fiducial")
+		(lib_id "Library:Fiducial")
 		(at 241.3 146.05 0)
 		(unit 1)
@@
 			)
 		)
-		(property "Footprint" "Fiducial:Fiducial_1mm_Mask2mm"
+		(property "Footprint" "Library:Fiducial_1mm_Mask2mm"
 			(at 241.3 146.05 0)
 			(effects
@@
 			)
 		)
-		(property "Footprint" "LED_SMD:LED_0603_1608Metric"
+		(property "Footprint" "Library:LED_0603_1608Metric"
 			(at 87.63 74.93 0)
 			(effects
@@
 			)
 		)
-		(property "Footprint" "Resistor_SMD:R_0402_1005Metric"
+		(property "Footprint" "Library:R_0402_1005Metric"
 			(at 98.044 73.914 90)
 			(effects
@@
 			)
 		)
-		(property "Footprint" "LED_SMD:LED_0603_1608Metric"
+		(property "Footprint" "Library:LED_0603_1608Metric"
 			(at 87.63 49.53 0)
 			(effects
@@
 			)
 		)
-		(property "Footprint" "Package_TO_SOT_SMD:SOT-23"
+		(property "Footprint" "Library:SOT-23"
 			(at 49.53 64.135 0)
 			(effects
@@
 			)
 		)
-		(property "Footprint" "LED_SMD:LED_0603_1608Metric"
+		(property "Footprint" "Library:LED_0603_1608Metric"
 			(at 87.63 36.83 0)
 			(effects

Commit message: minor changes
Parts:
- added J13: Polarity Select, Connector_PinHeader_2.54mm:PinHeader_2x02_P2.54mm_Vertical, symbol Connector_Generic:Conn_02x02_Top_Bottom
Connections:
- net +3.3V: now also J13.4 (Pin_4); no longer J8.2 (Pin_2)
- net GND: now also J13.1 (Pin_1); no longer J8.1 (Pin_1)
- new net T1: J13.3 (Pin_3), J8.1 (Pin_1)
- new net T2: J13.2 (Pin_2), J8.2 (Pin_2)
Other:
- moved on the sheet: J8
Changed lines of the file:
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@@
 	(wire
 		(pts
+			(xy 191.77 44.45) (xy 193.04 44.45)
+		)
+		(stroke
+			(width 0)
+			(type default)
+		)
+	)
+	(wire
+		(pts
 			(xy 186.69 63.5) (xy 186.69 66.04)
 		)
@@
 		)
 	)
+	(label "T1"
+		(at 173.99 46.99 0)
+		(effects
+			(font
+				(size 1.27 1.27)
+			)
+			(justify left bottom)
+		)
+	)
 	(label "GPIO10"
 		(at 175.26 132.08 180)
@@
 		)
 	)
+	(label "T2"
+		(at 173.99 44.45 0)
+		(effects
+			(font
+				(size 1.27 1.27)
+			)
+			(justify left bottom)
+		)
+	)
 	(label "GPIO11"
 		(at 175.26 134.62 180)
@@
 	)
 	(label "SDA"
-		(at 185.42 39.37 0)
+		(at 173.99 39.37 0)
 		(effects
 			(font
@@
 	)
 	(label "SCL"
-		(at 185.42 41.91 0)
+		(at 173.99 41.91 0)
 		(effects
 			(font
@@
 		)
 	)
+	(label "T2"
+		(at 205.74 44.45 0)
+		(effects
+			(font
+				(size 1.27 1.27)
+			)
+			(justify left bottom)
+		)
+	)
 	(label "GPIO19"
 		(at 77.47 137.16 0)
@@
 		)
 	)
+	(label "T1"
+		(at 193.04 46.99 180)
+		(effects
+			(font
+				(size 1.27 1.27)
+			)
+			(justify right bottom)
+		)
+	)
 	(label "GPIO11"
 		(at 41.91 134.62 180)
@@
 	)
 	(symbol
+		(lib_id "Connector_Generic:Conn_02x02_Top_Bottom")
+		(at 200.66 46.99 180)
+		(unit 1)
+		(exclude_from_sim no)
+		(in_bom yes)
+		(on_board yes)
+		(dnp no)
+		(property "Reference" "J13"
+			(at 198.374 40.64 0)
+			(effects
+				(font
+					(size 1.27 1.27)
+				)
+			)
+		)
+		(property "Value" "Polarity Select"
+			(at 198.882 38.354 0)
+			(effects
+				(font
+					(size 1.27 1.27)
+				)
+			)
+		)
+		(property "Footprint" "Connector_PinHeader_2.54mm:PinHeader_2x02_P2.54mm_Vertical"
+			(at 200.66 46.99 0)
+			(effects
+				(font
+					(size 1.27 1.27)
+				)
+				(hide yes)
+			)
+		)
+		(property "Datasheet" "~"
+			(at 200.66 46.99 0)
+			(effects
+				(font
+					(size 1.27 1.27)
+				)
+				(hide yes)
+			)
+		)
+		(property "Description" "Generic connector, double row, 02x02, top/bottom pin numbering scheme (row 1: 1...pins_per_row, row2: pins_per_row+1 ... num_pins), script generated (kicad-library-utils/schlib/autogen/connector/)"
+			(at 200.66 46.99 0)
+			(effects
+				(font
+					(size 1.27 1.27)
+				)
+				(hide yes)
+			)
+		)
+		(pin "1"
+		)
+		(pin "2"
+		)
+		(pin "4"
+		)
+		(pin "3"
+		)
+		(instances
+			(project "pico-breadboard"
+				(path "/8dc432d0-705f-48a2-b043-b7130b9baf7d"
+					(reference "J13")
+					(unit 1)
+				)
+			)
+		)
+	)
+	(symbol
 		(lib_id "Library:Conn_01x04")
 		(at 255.27 43.18 0)
@@
 	)
 	(symbol
-		(lib_id "Library:+3.3V")
-		(at 185.42 44.45 270)
-		(unit 1)
-		(exclude_from_sim no)
-		(in_bom yes)
-		(on_board yes)
-		(dnp no)
-		(fields_autoplaced yes)
-		(property "Reference" "#PWR019"
-			(at 181.61 44.45 0)
-			(effects
-				(font
-					(size 1.27 1.27)
-				)
-				(hide yes)
-			)
-		)
-		(property "Value" "+3.3V"
-			(at 189.23 44.4499 90)
-			(effects
-				(font
-					(size 1.27 1.27)
-				)
-				(justify left)
-			)
-		)
-		(property "Footprint" ""
-			(at 185.42 44.45 0)
-			(effects
-				(font
-					(size 1.27 1.27)
-				)
-				(hide yes)
-			)
-		)
-		(property "Datasheet" ""
-			(at 185.42 44.45 0)
-			(effects
-				(font
-					(size 1.27 1.27)
-				)
-				(hide yes)
-			)
-		)
-		(property "Description" "Power symbol creates a global label with name \"+3.3V\""
-			(at 185.42 44.45 0)
-			(effects
-				(font
-					(size 1.27 1.27)
-				)
-				(hide yes)
-			)
-		)
-		(pin "1"
-		)
-		(instances
-			(project "pico-breadboard"
-				(path "/8dc432d0-705f-48a2-b043-b7130b9baf7d"
-					(reference "#PWR019")
-					(unit 1)
-				)
-			)
-		)
-	)
-	(symbol
 		(lib_id "Library:SW_SPST")
 		(at 125.73 74.93 0)
@@
 	(symbol
 		(lib_id "Library:Conn_01x04")
-		(at 180.34 44.45 180)
+		(at 168.91 44.45 180)
 		(unit 1)
 		(exclude_from_sim no)
@@
 		(dnp no)
 		(property "Reference" "J8"
-			(at 177.8 44.4501 0)
+			(at 166.37 44.4501 0)
 			(effects
 				(font
@@
 		)
 		(property "Value" "SCREEN CONNECTOR"
-			(at 189.23 35.56 0)
+			(at 177.8 35.56 0)
 			(effects
 				(font
@@
 		)
 		(property "Footprint" "Library:PinHeader_1x04_P2.54mm_Vertical"
-			(at 180.34 44.45 0)
+			(at 168.91 44.45 0)
 			(effects
 				(font
@@
 		)
 		(property "Datasheet" "~"
-			(at 180.34 44.45 0)
+			(at 168.91 44.45 0)
 			(effects
 				(font
@@
 		)
 		(property "Description" "Generic connector, single row, 01x04, script generated (kicad-library-utils/schlib/autogen/connector/)"
-			(at 180.34 44.45 0)
+			(at 168.91 44.45 0)
 			(effects
 				(font
@@
 	)
 	(symbol
+		(lib_id "Library:GND")
+		(at 205.74 46.99 0)
+		(unit 1)
+		(exclude_from_sim no)
+		(in_bom yes)
+		(on_board yes)
+		(dnp no)
+		(fields_autoplaced yes)
+		(property "Reference" "#PWR12"
+			(at 205.74 53.34 0)
+			(effects
+				(font
+					(size 1.27 1.27)
+				)
+				(hide yes)
+			)
+		)
+		(property "Value" "GND"
+			(at 205.74 52.07 0)
+			(effects
+				(font
+					(size 1.27 1.27)
+				)
+			)
+		)
+		(property "Footprint" ""
+			(at 205.74 46.99 0)
+			(effects
+				(font
+					(size 1.27 1.27)
+				)
+				(hide yes)
+			)
+		)
+		(property "Datasheet" ""
+			(at 205.74 46.99 0)
+			(effects
+				(font
+					(size 1.27 1.27)
+				)
+				(hide yes)
+			)
+		)
+		(property "Description" "Power symbol creates a global label with name \"GND\" , ground"
+			(at 205.74 46.99 0)
+			(effects
+				(font
+					(size 1.27 1.27)
+				)
+				(hide yes)
+			)
+		)
+		(pin "1"
+		)
+		(instances
+			(project "pico-breadboard"
+				(path "/8dc432d0-705f-48a2-b043-b7130b9baf7d"
+					(reference "#PWR12")
+					(unit 1)
+				)
+			)
+		)
+	)
+	(symbol
 		(lib_id "Library:LED")
 		(at 87.63 62.23 180)
@@
 	)
 	(symbol
-		(lib_id "Library:GND")
-		(at 185.42 46.99 90)
+		(lib_id "Library:+3.3V")
+		(at 191.77 44.45 90)
 		(unit 1)
 		(exclude_from_sim no)
@@
 		(dnp no)
 		(fields_autoplaced yes)
-		(property "Reference" "#PWR020"
-			(at 191.77 46.99 0)
+		(property "Reference" "#PWR11"
+			(at 195.58 44.45 0)
 			(effects
 				(font
@@
 			)
 		)
-		(property "Value" "GND"
-			(at 189.23 46.9899 90)
+		(property "Value" "+3.3V"
+			(at 187.96 44.4499 90)
 			(effects
 				(font
 					(size 1.27 1.27)
 				)
-				(justify right)
+				(justify left)
 			)
 		)
 		(property "Footprint" ""
-			(at 185.42 46.99 0)
+			(at 191.77 44.45 0)
 			(effects
 				(font
@@
 		)
 		(property "Datasheet" ""
-			(at 185.42 46.99 0)
+			(at 191.77 44.45 0)
 			(effects
 				(font
@@
 			)
 		)
-		(property "Description" "Power symbol creates a global label with name \"GND\" , ground"
-			(at 185.42 46.99 0)
+		(property "Description" "Power symbol creates a global label with name \"+3.3V\""
+			(at 191.77 44.45 0)
 			(effects
 				(font
@@
 			(project "pico-breadboard"
 				(path "/8dc432d0-705f-48a2-b043-b7130b9baf7d"
-					(reference "#PWR020")
+					(reference "#PWR11")
 					(unit 1)
 				)
